Commit message: Change ros2_control and gazebo_conrol

File: description/gazebo_control.xacro (robot description, xacro)
@@ -4,10 +4,8 @@
         <plugin filename="gz-sim-joint-state-publisher-system" name="gz::sim::systems::JointStatePublisher">
             <topic>joint_states</topic>
-            <joint_name>front_left_steering_joint</joint_name>
-            <joint_name>front_right_steering_joint</joint_name>
-            <joint_name>front_left_wheel_joint</joint_name>
-            <joint_name>front_right_wheel_joint</joint_name>
-            <joint_name>rear_left_wheel_joint</joint_name>
-            <joint_name>rear_right_wheel_joint</joint_name>
+            <joint_name>front_steering_joint</joint_name>
+            <joint_name>rear_steering_joint</joint_name>
+            <joint_name>front_wheels_joint</joint_name>
+            <joint_name>rear_wheels_joint</joint_name>
         </plugin>
         <plugin filename="gz_ros2_control-system" name="gz_ros2_control::GazeboSimROS2ControlPlugin">

File: description/ros2_control.xacro (robot description, xacro)
@@ -5,6 +5,8 @@
             <hardware>
                 <plugin>diffdrive_arduino/DiffDriveArduino</plugin>
-                <param name="left_wheel_name">left_wheel_joint</param>
-                <param name="right_wheel_name">right_wheel_joint</param>
+                <param name="front_steering_name">front_steering_joint</param>
+                <param name="rear_steering_name">rear_steering_joint</param>
+                <param name="front_wheels_name">front_wheels_joint</param>
+                <param name="rear_wheels_name">rear_wheel_joint</param>
                 <param name="loop_rate">30</param>
                 <param name="device">/dev/ttyUSB0</param>
@@ -13,20 +15,38 @@
                 <param name="enc_counts_per_rev">3436</param>
             </hardware>
-            <joint name="left_wheel_joint">
-                <command_interface name="velocity">
-                    <param name="min">-10</param>
-                    <param name="max">10</param>
-                </command_interface>
-                <state_interface name="velocity"/>
-                <state_interface name="position"/>
-            </joint>
-            <joint name="right_wheel_joint">
-                <command_interface name="velocity">
-                    <param name="min">-10</param>
-                    <param name="max">10</param>
-                </command_interface>
-                <state_interface name="velocity"/>
-                <state_interface name="position"/>
-            </joint>
+        <joint name="front_steering_joint">
+            <command_interface name="position">
+                <param name="min">${-max_steering_angle}</param>
+                <param name="max">${max_steering_angle}</param>
+            </command_interface>
+            <state_interface name="position"/>
+            <state_interface name="effort"/>
+        </joint>
+        <joint name="rear_steering_joint">
+            <command_interface name="position">
+                <param name="min">${-max_steering_angle}</param>
+                <param name="max">${max_steering_angle}</param>
+            </command_interface>
+            <state_interface name="position"/>
+            <state_interface name="effort"/>
+        </joint>
+        <joint name="front_wheels_joint">
+            <command_interface name="velocity">
+                <param name="min">${-max_wheels_angular_velocity}</param>
+                <param name="max">${max_wheels_angular_velocity}</param>
+            </command_interface>
+            <state_interface name="position"/>
+            <state_interface name="velocity"/>
+            <state_interface name="effort"/>
+        </joint>
+        <joint name="rear_wheels_joint">
+            <command_interface name="velocity">
+                <param name="min">${-max_wheels_angular_velocity}</param>
+                <param name="max">${max_wheels_angular_velocity}</param>
+            </command_interface>
+            <state_interface name="position"/>
+            <state_interface name="velocity"/>
+            <state_interface name="effort"/>
+        </joint>
         </ros2_control>
     </xacro:unless>
