Commit message: Delete extra files and edit xacro files

File: description/robot.urdf.xacro (robot description, xacro)
@@ -68,6 +68,6 @@
     </collision>
   </link>
-  <!-- Chassis -->
-  <joint name="front_chassis_joint" type="revolute">
+  <!-- Steering -->
+  <joint name="front_steering_joint" type="revolute">
     <parent link="body_link"/>
     <child link="front_chassis_link"/>
@@ -76,5 +76,5 @@
     <limit effort="2000" lower="-0.5235987755982988" upper="0.5235987755982988" velocity="1"/>
   </joint>
-  <link name="front_chassis_link">
+  <link name="front_steering_link">
     <!-- <visual>
             <geometry></geometry>
@@ -85,33 +85,33 @@
         <cylinder length="0.225" radius="0.02"/>
       </geometry>
-      <material name="chassis"/>
-    </visual>
-    <visual>
-      <origin rpy="-1.5707963267948966 0 0" xyz="0 0.016575 0"/>
-      <geometry>
-        <cylinder length="0.03315" radius="0.0115"/>
-      </geometry>
-      <material name="chassis"/>
-    </visual>
-    <collision>
-      <geometry>
-        <cylinder length="0.225" radius="0.02"/>
-      </geometry>
-    </collision>
-    <collision>
-      <origin rpy="-1.5707963267948966 0 0" xyz="0 0.016575 0"/>
-      <geometry>
-        <cylinder length="0.03315" radius="0.0115"/>
-      </geometry>
-    </collision>
-  </link>
-  <joint name="rear_chassis_joint" type="revolute">
+      <material name="steering"/>
+    </visual>
+    <visual>
+      <origin rpy="-1.5707963267948966 0 0" xyz="0 0.016575 0"/>
+      <geometry>
+        <cylinder length="0.03315" radius="0.0115"/>
+      </geometry>
+      <material name="steering"/>
+    </visual>
+    <collision>
+      <geometry>
+        <cylinder length="0.225" radius="0.02"/>
+      </geometry>
+    </collision>
+    <collision>
+      <origin rpy="-1.5707963267948966 0 0" xyz="0 0.016575 0"/>
+      <geometry>
+        <cylinder length="0.03315" radius="0.0115"/>
+      </geometry>
+    </collision>
+  </link>
+  <joint name="rear_steering_joint" type="revolute">
     <parent link="body_link"/>
-    <child link="rear_chassis_link"/>
+    <child link="rear_steering_link"/>
     <origin rpy="1.5707963267948966 0 0" xyz="-0.19111999999999998 0 -0.07465000000000001"/>
     <axis xyz="0 -1 0"/>
     <limit effort="2000" lower="-0.5235987755982988" upper="0.5235987755982988" velocity="1"/>
   </joint>
-  <link name="rear_chassis_link">
+  <link name="rear_steering_link">
     <!-- <visual>
             <geometry></geometry>
@@ -122,12 +122,12 @@
         <cylinder length="0.225" radius="0.02"/>
       </geometry>
-      <material name="chassis"/>
-    </visual>
-    <visual>
-      <origin rpy="-1.5707963267948966 0 0" xyz="0 0.016575 0"/>
-      <geometry>
-        <cylinder length="0.03315" radius="0.0115"/>
-      </geometry>
-      <material name="chassis"/>
+      <material name="steering"/>
+    </visual>
+    <visual>
+      <origin rpy="-1.5707963267948966 0 0" xyz="0 0.016575 0"/>
+      <geometry>
+        <cylinder length="0.03315" radius="0.0115"/>
+      </geometry>
+      <material name="steering"/>
     </visual>
     <collision>
@@ -145,5 +145,5 @@
   <!-- Wheels -->
   <joint name="front_left_wheel_joint" type="continuous">
-    <parent link="front_chassis_link"/>
+    <parent link="front_steering_link"/>
     <child link="front_left_wheel_link"/>
     <origin rpy="-3.141592653589793 0 0" xyz="0 0 -0.135605"/>
@@ -168,5 +168,5 @@
   </link>
   <joint name="front_right_wheel_joint" type="continuous">
-    <parent link="front_chassis_link"/>
+    <parent link="front_steering_link"/>
     <child link="front_right_wheel_link"/>
     <origin xyz="0 0 0.135605"/>
@@ -191,5 +191,5 @@
   </link>
   <joint name="rear_left_wheel_joint" type="continuous">
-    <parent link="rear_chassis_link"/>
+    <parent link="rear_steering_link"/>
     <child link="rear_left_wheel_link"/>
     <origin rpy="-3.141592653589793 0 0" xyz="0 0 -0.135605"/>
@@ -214,5 +214,5 @@
   </link>
   <joint name="rear_right_wheel_joint" type="continuous">
-    <parent link="rear_chassis_link"/>
+    <parent link="rear_steering_link"/>
     <child link="rear_right_wheel_link"/>
     <origin xyz="0 0 0.135605"/>

File: description/ros2_control.xacro (robot description, xacro)
@@ -31,8 +31,8 @@
             <state_interface name="effort"/>
         </joint>
-        <joint name="front_wheels_joint">
+        <joint name="front_left_wheel_joint">
             <command_interface name="velocity">
-                <param name="min">${-max_wheels_angular_velocity}</param>
-                <param name="max">${max_wheels_angular_velocity}</param>
+                <param name="min">${-max_wheel_angular_velocity}</param>
+                <param name="max">${max_wheel_angular_velocity}</param>
             </command_interface>
             <state_interface name="position"/>
@@ -40,8 +40,26 @@
             <state_interface name="effort"/>
         </joint>
-        <joint name="rear_wheels_joint">
+        <joint name="front_right_wheel_joint">
             <command_interface name="velocity">
-                <param name="min">${-max_wheels_angular_velocity}</param>
-                <param name="max">${max_wheels_angular_velocity}</param>
+                <param name="min">${-max_wheel_angular_velocity}</param>
+                <param name="max">${max_wheel_angular_velocity}</param>
+            </command_interface>
+            <state_interface name="position"/>
+            <state_interface name="velocity"/>
+            <state_interface name="effort"/>
+        </joint>
+        <joint name="rear_left_wheel_joint">
+            <command_interface name="velocity">
+                <param name="min">${-max_wheel_angular_velocity}</param>
+                <param name="max">${max_wheel_angular_velocity}</param>
+            </command_interface>
+            <state_interface name="position"/>
+            <state_interface name="velocity"/>
+            <state_interface name="effort"/>
+        </joint>
+        <joint name="rear_right_wheel_joint">
+            <command_interface name="velocity">
+                <param name="min">${-max_wheel_angular_velocity}</param>
+                <param name="max">${max_wheel_angular_velocity}</param>
             </command_interface>
             <state_interface name="position"/>
@@ -56,9 +74,21 @@
             <plugin>gz_ros2_control/GazeboSimSystem</plugin>
         </hardware>
-        <joint name="front_left_steering_joint">
+        <joint name="front_steering_joint">
             <command_interface name="position">
                 <param name="min">${-max_steering_angle}</param>
                 <param name="max">${max_steering_angle}</param>
             </command_interface>
+            <state_interface name="position"/>
+            <state_interface name="effort"/>
+        </joint>
+        <joint name="rear_steering_joint">
+            <command_interface name="position">
+                <param name="min">${-max_steering_angle}</param>
+                <param name="max">${max_steering_angle}</param>
+            </command_interface>
+            <state_interface name="position"/>
+            <state_interface name="effort"/>
+        </joint>
+        <joint name="front_left_wheel_joint">
             <command_interface name="velocity">
                 <param name="min">${-max_wheel_angular_velocity}</param>
@@ -69,9 +99,5 @@
             <state_interface name="effort"/>
         </joint>
-        <joint name="front_right_steering_joint">
-            <command_interface name="position">
-                <param name="min">${-max_steering_angle}</param>
-                <param name="max">${max_steering_angle}</param>
-            </command_interface>
+        <joint name="front_right_wheel_joint">
             <command_interface name="velocity">
                 <param name="min">${-max_wheel_angular_velocity}</param>
@@ -83,8 +109,4 @@
         </joint>
         <joint name="rear_left_wheel_joint">
-            <command_interface name="position">
-                <param name="min">${-max_steering_angle}</param>
-                <param name="max">${max_steering_angle}</param>
-            </command_interface>
             <command_interface name="velocity">
                 <param name="min">${-max_wheel_angular_velocity}</param>
@@ -96,8 +118,4 @@
         </joint>
         <joint name="rear_right_wheel_joint">
-            <command_interface name="position">
-                <param name="min">${-max_steering_angle}</param>
-                <param name="max">${max_steering_angle}</param>
-            </command_interface>
             <command_interface name="velocity">
                 <param name="min">${-max_wheel_angular_velocity}</param>

Commit message: Some changes

File: description/robot.urdf.xacro (robot description, xacro)
@@ -6,14 +6,14 @@
 <robot name="robot">
   <material name="body">
-    <color rgba="0.05 0.05 0.05 1"/>
+    <color rgba="0.1 0.1 0.1 1"/>
   </material>
   <material name="bed">
-    <color rgba="0.05 0.05 0.05 1"/>
+    <color rgba="0.1 0.1 0.1 1"/>
   </material>
   <material name="chassis">
-    <color rgba="0.05 0.05 0.05 1"/>
+    <color rgba="0.1 0.1 0.1 1"/>
   </material>
   <material name="wheel">
-    <color rgba="0.05 0.05 0.05 1"/>
+    <color rgba="0.1 0.1 0.1 1"/>
   </material>
   <link name="base_link"/>
@@ -46,5 +46,5 @@
     <parent link="body_link"/>
     <child link="bed_link"/>
-    <origin xyz="-0.057 0 0.0965"/>
+    <origin xyz="-0.08200000000000002 0 0.0965"/>
   </joint>
   <link name="bed_link">
@@ -58,5 +58,5 @@
     <visual>
       <geometry>
-        <box size="0.47 0.27 0.11"/>
+        <box size="0.52 0.27 0.11"/>
       </geometry>
       <material name="bed"/>
@@ -64,20 +64,20 @@
     <collision>
       <geometry>
-        <box size="0.47 0.27 0.11"/>
-      </geometry>
-    </collision>
-  </link>
-  <!-- Steering -->
+        <box size="0.52 0.27 0.11"/>
+      </geometry>
+    </collision>
+  </link>
+  <!-- Chassis -->
   <joint name="front_steering_joint" type="revolute">
     <parent link="body_link"/>
-    <child link="front_chassis_link"/>
+    <child link="front_steering_link"/>
     <origin rpy="1.5707963267948966 0 0" xyz="0.0721 0 -0.07465000000000001"/>
     <axis xyz="0 -1 0"/>
-    <limit effort="2000" lower="-0.5235987755982988" upper="0.5235987755982988" velocity="1"/>
+    <limit effort="1" lower="-0.3490658503988659" upper="0.3490658503988659" velocity="1"/>
   </joint>
   <link name="front_steering_link">
     <!-- <visual>
             <geometry></geometry>
-            <material name="chassis"/>
+            <material name="steering"/>
         </visual> -->
     <visual>
@@ -111,10 +111,10 @@
     <origin rpy="1.5707963267948966 0 0" xyz="-0.19111999999999998 0 -0.07465000000000001"/>
     <axis xyz="0 -1 0"/>
-    <limit effort="2000" lower="-0.5235987755982988" upper="0.5235987755982988" velocity="1"/>
+    <limit effort="1" lower="-0.3490658503988659" upper="0.3490658503988659" velocity="1"/>
   </joint>
   <link name="rear_steering_link">
     <!-- <visual>
             <geometry></geometry>
-            <material name="chassis"/>
+            <material name="steering"/>
         </visual> -->
     <visual>

File: description/ros2_control.xacro (robot description, xacro)
@@ -7,6 +7,8 @@
                 <param name="front_steering_name">front_steering_joint</param>
                 <param name="rear_steering_name">rear_steering_joint</param>
-                <param name="front_wheels_name">front_wheels_joint</param>
-                <param name="rear_wheels_name">rear_wheel_joint</param>
+                <param name="front_left_wheel_name">front_left_wheel_joint</param>
+                <param name="front_right_wheel_name">front_right_wheel_joint</param>
+                <param name="rear_left_wheel_name">rear_left_wheel_joint</param>
+                <param name="rear_right_wheel_name">reae_right_wheel_joint</param>
                 <param name="loop_rate">30</param>
                 <param name="device">/dev/ttyUSB0</param>
